File: controller/analog.kicad_sch (KiCad schematic)
At the start: 0 parts

Commit message: Controller Complete
Completed Controller Section
Parts:
- added C32, C33, C34: C_Small, symbol Device:C_Small
- added J3: USB_A_Stacked, symbol Connector:USB_A_Stacked
- added J7: 68602-116HLF, CONN_68602-116HLF_AMP, symbol 2024-05-08_23-41-22:68602-116HLF
Connections:
- new net: J3.1 (VBUS1), J3.5 (VBUS2), J7.16
- new net +3.3V: C32.1, C33.1, C34.1, J7.1, J7.3, J7.5
- new net Ac_Voltage_In: J7.8
- new net Batt_Sense: J7.13
- new net Car_En: J7.12
- new net Charge_Status: J7.14
- new net Current_in: J7.7
- new net DC_i2c_scl: J7.9
- new net DC_i2c_sda: J7.10
- new net GND: C32.2, C33.2, C34.2, J3.4 (GND1), J3.8 (GND2), J3.9 (Shield), J7.2, J7.4, J7.6
- new net USBC_Vbus1: J7.15
- new net usbc_vbus2: J7.11
- no-connect marks 0 -> 4
Other:
- company: (none) -> Voltaworks
