File: controller/usb_C.kicad_sch (KiCad schematic)
At the start: 14 parts, among them J1 USB_C_Receptacle, J2 USB_C_Receptacle, U4 TPS65988DHRSHR

Commit message: Controller Complete
Completed Controller Section
Connections:
- net c1_cc1: now also J1.A5 (CC1)
- net D+1 renamed usbd+
- net D-1 renamed usbd-
- net Vbus2 renamed vbus2
- no-connect marks 27 -> 45
Other:
- company: (none) -> Voltaworks
Changed lines of the file:
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@@
 	(generator_version "8.0")
 	(paper "A4")
+	(title_block
+		(company "Voltaworks")
+	)
 	(junction
 		(at 167.64 134.62)
@@
 	)
 	(no_connect
+		(at 57.15 137.16)
+	)
+	(no_connect
+		(at 57.15 58.42)
+	)
+	(no_connect
 		(at 115.57 60.96)
 	)
@@
 	)
 	(no_connect
+		(at 57.15 134.62)
+	)
+	(no_connect
 		(at 115.57 86.36)
 	)
 	(no_connect
+		(at 57.15 127)
+	)
+	(no_connect
 		(at 115.57 78.74)
 	)
@@
 	)
 	(no_connect
+		(at 57.15 142.24)
+	)
+	(no_connect
 		(at 115.57 53.34)
 	)
 	(no_connect
+		(at 57.15 66.04)
+	)
+	(no_connect
 		(at 115.57 71.12)
 	)
@@
 	)
 	(no_connect
+		(at 57.15 81.28)
+	)
+	(no_connect
 		(at 191.77 81.28)
 	)
@@
 	)
 	(no_connect
+		(at 57.15 144.78)
+	)
+	(no_connect
 		(at 115.57 48.26)
 	)
@@
 	)
 	(no_connect
+		(at 57.15 91.44)
+	)
+	(no_connect
+		(at 57.15 88.9)
+	)
+	(no_connect
+		(at 57.15 152.4)
+	)
+	(no_connect
+		(at 57.15 68.58)
+	)
+	(no_connect
+		(at 57.15 149.86)
+	)
+	(no_connect
+		(at 167.64 127)
+	)
+	(no_connect
+		(at 57.15 83.82)
+	)
+	(no_connect
+		(at 57.15 119.38)
+	)
+	(no_connect
 		(at 115.57 50.8)
 	)
@@
 	(no_connect
 		(at 115.57 40.64)
+	)
+	(no_connect
+		(at 57.15 129.54)
+	)
+	(no_connect
+		(at 167.64 121.92)
 	)
 	(no_connect
@@
 	)
 	(label "c1_cc1"
-		(at 60.96 37.592 0)
+		(at 60.96 38.1 0)
 		(fields_autoplaced yes)
 		(effects
@@
 		(fields_autoplaced yes)
 		(effects
+			(font
+				(size 1.27 1.27)
+			)
+			(justify left)
+		)
+	)
+	(hierarchical_label "vbus2"
+		(shape input)
+		(at 111.76 121.92 180)
+		(fields_autoplaced yes)
+		(effects
+			(font
+				(size 1.27 1.27)
+			)
+			(justify right)
+		)
+	)
+	(hierarchical_label "usbd-"
+		(shape input)
+		(at 66.04 45.72 0)
+		(fields_autoplaced yes)
+		(effects
+			(font
+				(size 1.27 1.27)
+			)
+			(justify left)
+		)
+	)
+	(hierarchical_label "vbus1"
+		(shape input)
+		(at 111.76 114.3 180)
+		(fields_autoplaced yes)
+		(effects
+			(font
+				(size 1.27 1.27)
+			)
+			(justify right)
+		)
+	)
+	(hierarchical_label "usbd+"
+		(shape input)
+		(at 66.04 53.34 0)
+		(fields_autoplaced yes)
+		(effects
